File: cart/banana_proto/banana_proto.kicad_pcb (KiCad board)
At the start: 2 copper layers, 100 x 64.8 mm, 117 parts, among them Q1 2N3904, Q2 2N3904, U1 MT25QL01GBBB, U3 CS4334, U4 MAX4395, U6 NCP699SN50T1G

Commit message: pcb almost ready
Parts:
- removed R19: 560, Resistor_THT:R_Axial_DIN0207_L6.3mm_D2.5mm_P7.62mm_Horizontal
- added B1: Banana_PI_M2_Zero, BPI:BananaPI M2 Zero, F.Cu at (122.1, 66.9)
- added BUS1: MSX_SLOT_EDGE-CON, Footprints:msx_cartridge, F.Cu at (157.5, 130.0)
- added D35: BZT52C2V7-TP, Diode_SMD:D_SOD-123, F.Cu at (137.2, 115.8)
- added J2: COMPOSITE, Connector_PinHeader_2.54mm:PinHeader_1x01_P2.54mm_Vertical, F.Cu at (121.0, 71.7)
- added J3: AudioJack3_Ground, Connector_Audio:Jack_3.5mm_PJ320E_Horizontal, F.Cu at (102.9, 78.4)
- added U2: CartBus, Footprints:DSL_Cartridge_Reader, F.Cu at (152.4, 94.0)
- added U5: ILI9341_TFT_LCD_Module, BPI:ILI9341 TFT LCD 24 modul, F.Cu at (108.7, 69.1)
- C18: value 2200uF 6.3V Radial -> 2200uF 6.3V; moved to F.Cu
- D12, D14, R37, R39: moved to B.Cu
- R1, R2: value 6K -> 10k; footprint Resistor_THT:R_Axial_DIN0207_L6.3mm_D2.5mm_P7.62mm_Horizontal -> Resistor_SMD:R_0805_2012Metric
- R10, R11: value 267k -> 10k; footprint Resistor_THT:R_Axial_DIN0207_L6.3mm_D2.5mm_P7.62mm_Horizontal -> Resistor_SMD:R_0805_2012Metric
- R15, R16: value 10k -> 560; footprint Resistor_THT:R_Axial_DIN0207_L6.3mm_D2.5mm_P7.62mm_Horizontal -> Resistor_SMD:R_0805_2012Metric
- R17: footprint Resistor_THT:R_Axial_DIN0207_L6.3mm_D2.5mm_P7.62mm_Horizontal -> Resistor_SMD:R_0805_2012Metric
- R18: value 560 -> 330; footprint Resistor_THT:R_Axial_DIN0207_L6.3mm_D2.5mm_P7.62mm_Horizontal -> Resistor_SMD:R_0805_2012Metric
- R5, R6: value 10k -> 267K; footprint Resistor_THT:R_Axial_DIN0207_L6.3mm_D2.5mm_P7.62mm_Horizontal -> Resistor_SMD:R_0805_2012Metric
- moved C10 211.7 mm to (174.2, 80.0), turned to 90 degrees
- moved C1 205.8 mm to (194.1, 100.6), turned to 180 degrees
- moved C3 204.6 mm to (199.6, 95.7), turned to -90 degrees
- moved R4 193.2 mm to (174.3, 87.8), turned to -90 degrees
- moved R18 190.7 mm to (137.2, 121.7), turned to -90 degrees
- moved R3 186.9 mm to (191.1, 78.8), turned to 90 degrees
- moved U1 186.3 mm to (182.7, 84.2), turned to 90 degrees
- moved C2 181.5 mm to (148.8, 104.1), turned to 180 degrees
- moved R7 174.5 mm to (120.9, 96.5), turned to 180 degrees
- moved R17 171.4 mm to (117.6, 93.0), turned to 90 degrees
- moved C7 168.8 mm to (121.4, 80.5), turned to 90 degrees
- moved D1 168.6 mm to (119.9, 113.5), turned to 90 degrees
- moved C18 164.1 mm to (200.0, 118.4), turned to 180 degrees
- moved R14 161.4 mm to (122.9, 105.9), turned to -90 degrees
- moved R9 161.2 mm to (120.9, 102.6), turned to 180 degrees
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Connections:
- R1 pad 1: GND -> +5VA
- R1 pad 2: Net-(J1-Pad5) -> Net-(R1-Pad2)
- R10 pad 1: GND -> Net-(C11-Pad2)
- R10 pad 2: /SND_R_RAW -> GND
- R11 pad 1: GND -> Net-(C12-Pad2)
- R11 pad 2: /SND_L_RAW -> GND
- R15 pad 1: GND -> /SPKR_R
- R16 pad 1: GND -> /SPKR_L
- R17 pad 1: Net-(C11-Pad2) -> /SND
- R17 pad 2: /SPKR_R -> Net-(R17-Pad2)
- R18 pad 1: Net-(C12-Pad2) -> /_~{SYS_CLK}
- R18 pad 2: /SPKR_L -> /SYS_CLK
- R2 pad 1: GND -> Net-(R1-Pad2)
- R2 pad 2: Net-(J1-Pad4) -> GND
- R5 pad 1: Net-(R5-Pad1) -> /SND_R_RAW
- R5 pad 2: +5VA -> GND
- R6 pad 1: GND -> /SND_L_RAW
- R6 pad 2: Net-(R5-Pad1) -> GND
- U3 pad 2: Net-(R5-Pad1) -> Net-(R1-Pad2)
- U4 pad 1: Net-(R21-Pad1) -> Net-(R13-Pad1)
- U4 pad 10: /SND_L_RAW -> /SND_R_RAW
- U4 pad 13: Net-(R19-Pad1) -> Net-(R17-Pad2)
- U4 pad 14: Net-(R19-Pad1) -> Net-(R17-Pad2)
- U4 pad 2: Net-(R21-Pad1) -> Net-(R13-Pad1)
- U4 pad 3: Net-(R20-Pad2) -> /SND_L_RAW
- U4 pad 5: /SND_R_RAW -> Net-(R20-Pad2)
- U4 pad 6: Net-(R12-Pad2) -> Net-(R21-Pad1)
- U4 pad 7: Net-(R12-Pad2) -> Net-(R21-Pad1)
- U4 pad 8: Net-(R13-Pad1) -> Net-(R12-Pad2)
- U4 pad 9: Net-(R13-Pad1) -> Net-(R12-Pad2)
Routing:
- net +5V: track 0.00 -> 154.6 mm, vias 0 -> 1
- net /SPI0_MISO: track 0.00 -> 125.7 mm, vias 0 -> 1
- net /SPI0_CLK: track 0.00 -> 110.5 mm, vias 0 -> 1
- net /SPI0_MOSI: track 0.00 -> 109.3 mm, vias 0 -> 1
- net /_A4: track 0.00 -> 87.3 mm, vias 0 -> 2
- net /_A5: track 0.00 -> 87.3 mm, vias 0 -> 3
- net /_A15: track 0.00 -> 75.4 mm, vias 0 -> 1
- net +5VA: track 0.00 -> 72.6 mm
- net /LCD_~{CS}: track 0.00 -> 72.3 mm
- net /LCD_~{RESET}: track 0.00 -> 69.8 mm
- net /LCD_D/~{C}: track 0.00 -> 67.3 mm
- net GND: track 0.00 -> 65.9 mm, vias 0 -> 168
- net /_A6: track 0.00 -> 58.1 mm, vias 0 -> 1
- net /_A11: track 0.00 -> 56.9 mm, vias 0 -> 1
- net /I2S_MCLK: track 0.00 -> 55.2 mm
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- added copper zone on In1.Cu, net +3V3
- added copper zone on B.Cu, net GND
- added copper zone on F.Cu, net GND
- added copper zone on In2.Cu, net GND
Other:
- board size 100 x 64.8 mm -> 101.6 x 65 mm
- copper layers 2 -> 4

Commit message: updated hal
Connections:
- B1 pad PAD0: GND -> (no net)
- B1 pad PAD1: GND -> (no net)
Routing:
- net /_~{SLTSL}: track 54.6 -> 52.3 mm
- net /_~{BUSDIR}: track 55.2 -> 53.1 mm
- net /_~{M1}: track 42.8 -> 40.8 mm
- net /_~{RFSH}: track 47.3 -> 45.3 mm
- net /_~{RESET}: track 46.3 -> 46.9 mm
- net /_~{WR}: track 45.0 -> 45.5 mm
