File: cart/banana_proto/banana_proto.kicad_sch (KiCad schematic)
At the start: 124 parts, among them J1 RJ45_Abracon_ARJP11A-MASA-B-A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, J2 COMPOSITE, J3 AudioJack3_Ground, Q1 2N3904, Q2 2N3904, U1 MT25QL01GBBB, U2 CartBus, U3 CS4334, U4 MAX4395, U5 ILI9341_TFT_LCD_Module, U6 NCP699SN50T1G

Commit message: pcb almost ready
Parts:
- removed J1: RJ45_Abracon_ARJP11A-MASA-B-A-EMU2, Connector_RJ:RJ45_Abracon_ARJP11A-MA_Horizontal, symbol Connector:RJ45_Abracon_ARJP11A-MASA-B-A-EMU2
- removed R19: 560, Resistor_THT:R_Axial_DIN0207_L6.3mm_D2.5mm_P7.62mm_Horizontal, symbol Device:R_US
- added D35: BZT52C2V7-TP, Diode_SMD:D_SOD-123, symbol Device:D_Zener
- C18: value 2200uF 6.3V Radial -> 2200uF 6.3V
- R1, R2: value 6K -> 10k; footprint Resistor_THT:R_Axial_DIN0207_L6.3mm_D2.5mm_P7.62mm_Horizontal -> Resistor_SMD:R_0805_2012Metric
- R10, R11: value 267k -> 10k; footprint Resistor_THT:R_Axial_DIN0207_L6.3mm_D2.5mm_P7.62mm_Horizontal -> Resistor_SMD:R_0805_2012Metric
- R15, R16: value 10k -> 560; footprint Resistor_THT:R_Axial_DIN0207_L6.3mm_D2.5mm_P7.62mm_Horizontal -> Resistor_SMD:R_0805_2012Metric
- R17: footprint Resistor_THT:R_Axial_DIN0207_L6.3mm_D2.5mm_P7.62mm_Horizontal -> Resistor_SMD:R_0805_2012Metric
- R18: value 560 -> 330; footprint Resistor_THT:R_Axial_DIN0207_L6.3mm_D2.5mm_P7.62mm_Horizontal -> Resistor_SMD:R_0805_2012Metric
- R5, R6: value 10k -> 267K; footprint Resistor_THT:R_Axial_DIN0207_L6.3mm_D2.5mm_P7.62mm_Horizontal -> Resistor_SMD:R_0805_2012Metric
- U4: footprint (none) -> Package_SO:TSSOP-14_4.4x5mm_P0.65mm
Connections:
- net _~{RFSH} / PL2 is gone; now on net _~{M1}: B1.P32 (PL2)
- net +2V8: no longer B1.C04 (VCC-2V8), B1.C24 (VCC-2V8)
- net +3V3: no longer U2.18 (A12)
- net +5VA: now also R1.1; no longer R5.2
- net A0: no longer U2.6 (A0)
- net A1: no longer U2.7 (A1)
- net A2: no longer U2.8 (A2)
- net A3: no longer U2.9 (A3)
- net A4: no longer U2.10 (A4)
- net A5: no longer U2.11 (A5)
- net A6: no longer U2.12 (A6)
- net A7: no longer U2.13 (A7)
- net COMPOSITE: now also J3.R2; no longer J3.S
- net D0: no longer U2.22 (D0)
- net D1: no longer U2.23 (D1)
- net D2: no longer U2.24 (D2)
- net D3: no longer U2.25 (D3)
- net D4: no longer U2.26 (D4)
- net D5: no longer U2.27 (D5)
- net D6: no longer U2.28 (D6)
- net D7: no longer U2.29 (D7)
- net GND: now also J3.R1, R10.2, R11.2, R2.2, R5.2, R6.2, D35.2 (A); no longer J3.R, R1.1, R10.1, R11.1, R15.1, R16.1, R2.1, R6.1
- net IRQ: now also B1.P26 (PC7); no longer B1.C16 (PE9)
- net PC4: no longer B1.P18 (PC4), U2.19 (A13)
- net PC7: no longer B1.P26 (PC7), U2.20 (A14), U5.3 (LCD_~{CS})
- net PE12: no longer B1.C05 (PE12), U5.5 (LCD_D/~{C})
- net SND: now also R17.1; no longer U2.31 (SND)
- net SND_L_RAW: now also R6.1, U4.3 (+); no longer R11.2, U4.10 (+)
- net SND_R_RAW: now also R5.1, U4.10 (+); no longer R10.2, U4.5 (+)
- net SPI0_CLK: no longer U2.16 (A10)
- net SPI0_CS: no longer U2.17 (A11)
- net SPI0_MISO: no longer U2.15 (A9)
- net SPI0_MOSI: no longer U2.14 (A8)
- net SPKR_L: now also R16.1; no longer R18.2
- net SPKR_R: now also J3.S, R15.1; no longer J3.G, R17.2
- net SYS_CLK: now also R18.2; no longer U2.2 (CLK~{})
- net WAIT: now also B1.P18 (PC4); no longer B1.C18 (PE8)
- net _~{BUSDIR}: now also B1.C08 (PE15); no longer B1.C14 (PE10)
- net _~{IORQ}: now also B1.C03 (PE13); no longer B1.C06 (PE14)
- net _~{M1} / PL4: no longer B1.P36 (PL4), U5.4 (LCD_~{RESET})
- net _~{MERQ}: now also B1.C05 (PE12); no longer B1.C08 (PE15)
- net _~{RESET}: now also B1.C06 (PE14); no longer B1.C12 (PE11)
- net _~{RFSH}: now also B1.P36 (PL4)
- net ~{IORQ}: no longer U2.5 (CS)
- net ~{RD}: no longer U2.4 (RD)
- net ~{RESET}: no longer U2.30 (RST)
- net ~{WR}: no longer U2.3 (WR)
- net at U4.6 (-), U4.7: now also R21.1; no longer R12.2
- net at C11.2, R15.2: now also R10.1; no longer R17.1
- net at C12.2, R16.2: now also R11.1; no longer R18.1
- net at U4.8, U4.9 (-): now also R12.2; no longer R13.1
- net at R20.2: now also U4.5 (+); no longer U4.3 (+)
- net at R1.2: now also R2.1, U3.2 (~{DEM}/SCLK)
- net at U4.13 (-), U4.14: now also R17.2
- net at U4.1, U4.2 (-): now also R13.1; no longer R21.1
- net PE13: no longer names the net of U2.21 (A15)
- net PE13: no longer B1.C03 (PE13)
- new net LCD_D/~{C}: B1.C14 (PE10), U5.5 (LCD_D/~{C})
- new net LCD_~{CS}: B1.C18 (PE8), U5.3 (LCD_~{CS})
- new net LCD_~{RESET}: B1.C16 (PE9), U5.4 (LCD_~{RESET})
- new net _~{SYS_CLK}: B1.C12 (PE11), D35.1 (K), R18.1
Other:
- moved on the sheet: D10, D2, D3, D4, D5, D6, D7, D8, D9, R27, R28, R29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

Commit message: updated hal
Parts:
- U2: value CartBus -> GBC Connector GNI17200
- U5: value ILI9341_TFT_LCD_Module -> ILI9341_TFT_LCD_Module MSP2402
Connections:
- net +3V3: now also U2.5 (CS)
- net GND: now also U2.21 (A15)
- net SPI0_CLK: now also U2.9 (A3), U5.10 (T_CLK)
- net SPI0_MISO: now also U2.7 (A1), U5.13 (T_DO)
- net SPI0_MOSI: now also U2.11 (A5), U5.12 (T_DIN)
- net _~{M1}: now also U2.15 (A9), U5.11 (T_CS)
- net _~{RESET}: now also U2.13 (A7), U2.19 (A13)
- net _~{RFSH}: now also U2.17 (A11)

Commit message: seems quite nice
Parts:
- C18: MPN (none) -> 6.3ZLH2200MEFC10X20
- C4: MPN (none) -> CL31F106ZPHNNNE; Mouser (none) -> CL31F106ZPHNNNE
- C7, C8: MPN (none) -> C1206C104K5RAC7210
- D10, D11, D12, D13, D14, D15, D16, D17, D18, D19, D2, D20, D21, D22, D23, D24, D25, D26, D27, D28, D29, D3, D30, D31, D32, D33, D34, D35, D4, D5, D6, D7, D8, D9: MPN (none) -> BZT52C2V7-TP; Mouser (none) -> BZT52C2V7-TP
- J3: MPN (none) -> PJ320E
- Q1, Q2: MPN (none) -> 2721-2N3904-ND; Mouser (none) -> 637-2N3904
- R18, R23, R24, R27, R28, R29, R3, R30, R31, R32, R33, R34, R35, R36, R37, R38, R39, R4, R40, R41, R42, R43, R44, R45, R46, R47, R48, R49, R50, R51, R52, R53, R54, R55, R56, R57, R58, R59: Mouser (none) -> CR0805-FX-3300ELF
